Commit message: new net

File: urdf/robomaster_ep_arm.urdf.xacro (robot description, xacro)
@@ -3,4 +3,5 @@
   <!--xacro:include filename="$(find robomaster_description)/urdf/robomaster_ep.gazebo.xacro"/-->
   <xacro:arg name="name" default=""/>
+  <xacro:arg name="camera_name" default=""/>
   <xacro:property name="_name" value="$(arg name)"/>
   <xacro:if value="${_name != ''}">
@@ -18,5 +19,5 @@
   <xacro:include filename="intelligent_controller.urdf.xacro"/>
   <xacro:include filename="extension.urdf.xacro"/>
-  <xacro:include filename="box.urdf.xacro"/>
+<!--  <xacro:include filename="box.urdf.xacro"/>-->
   <xacro:include filename="$(find robot_arm_description)/urdf/robot_arm.xacro"/>
   <!--xacro:include filename="sensor.urdf.xacro"/-->
@@ -24,5 +25,5 @@
   <xacro:base tf_prefix="${tf_prefix}"/>
   <xacro:extension tf_prefix="${tf_prefix}" use_rear_extension="true"/>
-  <xacro:box_ex tf_prefix="${tf_prefix}"/>
+<!--  <xacro:box_ex tf_prefix="${tf_prefix}"/>-->
   <xacro:intelligent_controller tf_prefix="${tf_prefix}" mount="extension"/>
   <gazebo>
@@ -35,8 +36,15 @@
     </plugin>
   </gazebo>
-  <!-- d435  frame definition can be found at https://github.com/IntelRealSense/librealsense/blob/master/doc/d435i.md
-  <xacro:include filename="$(find realsense_gazebo_description)/urdf/_d435_0.urdf.xacro"/>
-  <xacro:sensor_d435_0  parent="box_base_link" name="D435_camera_0" topics_ns="D435_camera_0" visualize="true">
-    <origin xyz="0.12 0 0.035" rpy="0.0 0.0 0.0"/>
-  </xacro:sensor_d435_0> -->
+  <xacro:include filename="demo_camera.urdf.xacro"/>
+  <xacro:camera_macro camera_name="$(arg camera_name)"
+                    image_topic="/$(arg camera_name)/image_raw"
+                    camera_info_topic="/$(arg camera_name)/camera_info" />
+<!--&lt;!&ndash;   d435  frame definition can be found at https://github.com/IntelRealSense/librealsense/blob/master/doc/d435i.md&ndash;&gt;-->
+<!--  <xacro:include filename="$(find realsense_gazebo_description)/urdf/_d435i.urdf.xacro"/>-->
+<!--  <xacro:sensor_d435i parent="box_base_link" name="D435i_camera_$(arg camera_name)" topics_ns="$(arg camera_name)" visualize="true">-->
+<!--    <origin xyz="0.12 0 0.035" rpy="1.57 -0.785 0.0"/>-->
+<!--  </xacro:sensor_d435i>-->
+<!--  <xacro:sensor_d435i parent="box_base_link" name="D435i_camera_$(arg camera_name)" topics_ns="$(arg camera_name)" visualize="true">-->
+<!--    <origin xyz="0.12 0 0.035" rpy="1.57 -0.785 0.0"/>-->
+<!--  </xacro:sensor_d435i>-->
 </robot>
